Commit message: robot in gazebo

File: description/robot_core.xacro (robot description, xacro)
@@ -42,6 +42,9 @@
         </xacro:inertial_box>
     </link>
+    <gazebo reference="chassis_link">
+        <material>Gazebo/White</material>
+    </gazebo>
     <!-- LEFT WHEEL -->
-    <joint name="left_wheel_link" type="continuous">
+    <joint name="left_wheel_joint" type="continuous">
         <parent link="base_link"/>
         <child link="left_wheel_link"/>
@@ -65,6 +68,9 @@
         </xacro:inertial_cylinder>
     </link>
+    <gazebo reference="left_wheel_link">
+        <material>Gazebo/Blue</material>
+    </gazebo>
     <!-- RIGHT WHEEL -->
-    <joint name="right_wheel_link" type="continuous">
+    <joint name="right_wheel_joint" type="continuous">
         <parent link="base_link"/>
         <child link="right_wheel_link"/>
@@ -88,6 +94,9 @@
         </xacro:inertial_cylinder>
     </link>
+    <gazebo reference="right_wheel_link">
+        <material>Gazebo/Blue</material>
+    </gazebo>
     <!-- CASTER WHEEL -->
-    <joint name="caster_wheel_join" type="fixed">
+    <joint name="caster_wheel_joint" type="fixed">
         <parent link="chassis_link"/>
         <child link="caster_wheel_link"/>
@@ -111,3 +120,6 @@
         </xacro:inertial_sphere>
     </link>
+    <gazebo reference="caster_wheel_link">
+        <material>Gazebo/Black</material>
+    </gazebo>
 </robot>
